File: Sensor_Unit/9v_battery.kicad_sch (KiCad schematic)
At the start: 4 parts, among them SW2 SLW-1276864-4A-D

Commit message: Week 11 Sensor Unit Final Design - Submitted to Pinecone
Parts:
- added TP1: GND, TestPoint:TestPoint_Loop_D2.54mm_Drill1.5mm_Beaded, symbol Connector:TestPoint
- TP2: renamed from TP1; value TestPoint -> 9V; footprint (none) -> TestPoint:TestPoint_Loop_D2.54mm_Drill1.5mm_Beaded
Connections:
- net GND: now also TP1.1
Other:
- moved on the sheet: TP2
Changed lines of the file:
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@@
 	)
 	(junction
-		(at 110.49 67.31)
+		(at 109.22 67.31)
 		(diameter 0)
 		(color 0 0 0 0)
@@
 		(color 0 0 0 0)
 	)
-	(wire
-		(pts
-			(xy 105.41 67.31) (xy 110.49 67.31)
+	(junction
+		(at 116.84 107.95)
+		(diameter 0)
+		(color 0 0 0 0)
+	)
+	(wire
+		(pts
+			(xy 105.41 67.31) (xy 109.22 67.31)
 		)
 		(stroke
@@
 	(wire
 		(pts
-			(xy 110.49 67.31) (xy 119.38 67.31)
-		)
-		(stroke
-			(width 0)
-			(type default)
-		)
-	)
-	(wire
-		(pts
 			(xy 116.84 107.95) (xy 105.41 107.95)
 		)
@@
 		(pts
 			(xy 105.41 62.23) (xy 105.41 67.31)
+		)
+		(stroke
+			(width 0)
+			(type default)
+		)
+	)
+	(wire
+		(pts
+			(xy 109.22 67.31) (xy 119.38 67.31)
 		)
 		(stroke
@@
 				(path "/631e2aad-29d7-4d5a-947a-1d7179af816f/55fbc23f-8772-4f41-8c66-e690c0637b4d"
 					(reference "#PWR091")
+					(unit 1)
+				)
+			)
+		)
+	)
+	(symbol
+		(lib_id "Connector:TestPoint")
+		(at 116.84 107.95 270)
+		(unit 1)
+		(exclude_from_sim no)
+		(in_bom yes)
+		(on_board yes)
+		(dnp no)
+		(fields_autoplaced yes)
+		(property "Reference" "TP1"
+			(at 121.92 106.6799 90)
+			(effects
+				(font
+					(size 1.27 1.27)
+				)
+				(justify left)
+			)
+		)
+		(property "Value" "GND"
+			(at 121.92 109.2199 90)
+			(effects
+				(font
+					(size 1.27 1.27)
+				)
+				(justify left)
+			)
+		)
+		(property "Footprint" "TestPoint:TestPoint_Loop_D2.54mm_Drill1.5mm_Beaded"
+			(at 116.84 113.03 0)
+			(effects
+				(font
+					(size 1.27 1.27)
+				)
+				(hide yes)
+			)
+		)
+		(property "Datasheet" "~"
+			(at 116.84 113.03 0)
+			(effects
+				(font
+					(size 1.27 1.27)
+				)
+				(hide yes)
+			)
+		)
+		(property "Description" "test point"
+			(at 116.84 107.95 0)
+			(effects
+				(font
+					(size 1.27 1.27)
+				)
+				(hide yes)
+			)
+		)
+		(pin "1"
+		)
+		(instances
+			(project "Sensor_Unit"
+				(path "/631e2aad-29d7-4d5a-947a-1d7179af816f/55fbc23f-8772-4f41-8c66-e690c0637b4d"
+					(reference "TP1")
 					(unit 1)
 				)
@@
 	(symbol
 		(lib_id "Connector:TestPoint")
-		(at 110.49 67.31 0)
+		(at 109.22 67.31 0)
 		(unit 1)
 		(exclude_from_sim no)
@@
 		(dnp no)
 		(fields_autoplaced yes)
-		(property "Reference" "TP1"
-			(at 113.03 62.7379 0)
+		(property "Reference" "TP2"
+			(at 111.76 62.7379 0)
 			(effects
 				(font
@@
 			)
 		)
-		(property "Value" "TestPoint"
-			(at 113.03 65.2779 0)
+		(property "Value" "9V"
+			(at 111.76 65.2779 0)
 			(effects
 				(font
@@
 			)
 		)
-		(property "Footprint" ""
-			(at 115.57 67.31 0)
+		(property "Footprint" "TestPoint:TestPoint_Loop_D2.54mm_Drill1.5mm_Beaded"
+			(at 114.3 67.31 0)
 			(effects
 				(font
@@
 		)
 		(property "Datasheet" "~"
-			(at 115.57 67.31 0)
+			(at 114.3 67.31 0)
 			(effects
 				(font
@@
 		)
 		(property "Description" "test point"
-			(at 110.49 67.31 0)
+			(at 109.22 67.31 0)
 			(effects
 				(font
@@
 			(project "Sensor_Unit"
 				(path "/631e2aad-29d7-4d5a-947a-1d7179af816f/55fbc23f-8772-4f41-8c66-e690c0637b4d"
-					(reference "TP1")
+					(reference "TP2")
 					(unit 1)
 				)
