File: Sensor_Unit/Optical_Link_Sensor.kicad_sch (KiCad schematic)
At the start: 16 parts, among them J4 Conn_01x03_Pin, J5 Conn_01x03_Pin, J6 Conn_01x04_Pin, J7 Conn_01x05_Pin, Q1 2N3904, Q2 IRF9540N, Q3 2N3904

Commit message: Week 11 Sensor Unit Final Design - Submitted to Pinecone
Changed lines of the file:
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@@
 		(color 0 0 0 0)
 	)
-	(bus_entry
-		(at 228.6 60.96)
-		(size 2.54 2.54)
-		(stroke
-			(width 0)
-			(type default)
-		)
-	)
-	(bus_entry
-		(at 228.6 57.15)
-		(size 2.54 2.54)
-		(stroke
-			(width 0)
-			(type default)
-		)
-	)
 	(wire
 		(pts
@@
 		)
 	)
-	(bus
-		(pts
-			(xy 228.6 57.15) (xy 228.6 55.88)
-		)
-		(stroke
-			(width 0)
-			(type default)
-		)
-	)
-	(wire
-		(pts
-			(xy 231.14 63.5) (xy 233.68 63.5)
-		)
-		(stroke
-			(width 0)
-			(type default)
-		)
-	)
 	(wire
 		(pts
@@
 		)
 	)
-	(bus
-		(pts
-			(xy 228.6 60.96) (xy 228.6 57.15)
-		)
-		(stroke
-			(width 0)
-			(type default)
-		)
-	)
 	(wire
 		(pts
@@
 		)
 	)
-	(bus
-		(pts
-			(xy 228.6 55.88) (xy 226.06 55.88)
-		)
-		(stroke
-			(width 0)
-			(type default)
-		)
-	)
 	(wire
 		(pts
@@
 		(pts
 			(xy 60.96 116.84) (xy 73.66 116.84)
-		)
-		(stroke
-			(width 0)
-			(type default)
-		)
-	)
-	(wire
-		(pts
-			(xy 231.14 59.69) (xy 233.68 59.69)
 		)
 		(stroke
@@
 		)
 	)
-	(hierarchical_label "OPTIC_LINK"
-		(shape bidirectional)
-		(at 226.06 55.88 180)
-		(effects
-			(font
-				(size 1.27 1.27)
-			)
-			(justify right)
-		)
-	)
