File: Sensor_Unit/Power_Supply_Subsystem_+-15V.kicad_sch (KiCad schematic)
At the start: 32 parts, among them U10 NJU7662D-ND, U11 LM7905_TO220, U12 TL072, U13 AMS1117-3.3, U7 AP3012KTR-G1, U8 LM340T-15/NOPB, U9 LM7805_TO220

Commit message: Week 11 Sensor Unit Final Design - Submitted to Pinecone
Parts:
- added TP10: -1V65, TestPoint:TestPoint_Loop_D2.54mm_Drill1.5mm_Beaded, symbol Connector:TestPoint
- added TP3: 17V, TestPoint:TestPoint_Loop_D2.54mm_Drill1.5mm_Beaded, symbol Connector:TestPoint
- added TP4: 15V, TestPoint:TestPoint_Loop_D2.54mm_Drill1.5mm_Beaded, symbol Connector:TestPoint
- added TP5: -15V, TestPoint:TestPoint_Loop_D2.54mm_Drill1.5mm_Beaded, symbol Connector:TestPoint
- added TP6: 5V, TestPoint:TestPoint_Loop_D2.54mm_Drill1.5mm_Beaded, symbol Connector:TestPoint
- added TP7: -5V, TestPoint:TestPoint_Loop_D2.54mm_Drill1.5mm_Beaded, symbol Connector:TestPoint
- added TP8: 3V3, TestPoint:TestPoint_Loop_D2.54mm_Drill1.5mm_Beaded, symbol Connector:TestPoint
- added TP9: 1V65, TestPoint:TestPoint_Loop_D2.54mm_Drill1.5mm_Beaded, symbol Connector:TestPoint
- C20: value 10u -> 1u; Field5 10uF -> 1uF
- C21: value 22uF -> 2.2uF
Connections:
- net +15V: now also TP4.1
- net +3V3: now also TP8.1
- net +5V: now also TP6.1
- net -15V: now also C21.1, U11.2 (VI), TP5.1; no longer C20.1, U11.3 (VO)
- net -1V65: now also TP10.1
- net -5V: now also C20.1, U11.3 (VO), TP7.1; no longer C21.1, U11.2 (VI)
- net 17V: now also TP3.1
- net 1V65: now also TP9.1
