File: Sensor_Unit/Sensor_Unit.kicad_sch (KiCad schematic)
At the start: 0 parts

Commit message: Week 11 Sensor Unit Final Design - Submitted to Pinecone
Other:
- sheet Acce and Temp Sensor ports: added none; removed  TEMP_SENSOR, ACCE_SENSOR
- sheet Optical Link ports: added none; removed OPTIC_LINK
- sheet Peripherals ports: added none; removed ALARM_LED_ARRAYS
- sheet Sensor MCU ports: added none; removed  TEMP_SENSOR, ACCE_SENSOR, ALARM_LED_ARRAYS, JLink Header, OPTIC_LINK, PC_COM
- sheet Xiao and Jlink ports: added none; removed JLink Header, PC_COM
