File: Sensor_Unit/Xiao_Jlink.kicad_sch (KiCad schematic)
At the start: 6 parts, among them J1 ETSG: 07-20-01, SW1 S201031MS02Q, U2 SeeeduinoXIAO

Commit message: Week 11 Sensor Unit Final Design - Submitted to Pinecone
Parts:
- removed C8, C9: 10u, Capacitor_SMD:C_0805_2012Metric_Pad1.18x1.45mm_HandSolder, symbol Device:C
- removed D1: 7.5V 500mW 5%, kicad_footprint-library-engg3800-alvin:DIOAD928W47L399D179, symbol Earr_loggy_sym_lib:BZX79C7V5
- removed SW1: S201031MS02Q, kicad_footprint-library-engg3800-alvin:SW6_S201031MS02Q_CNK, symbol Earr_loggy_sym_lib:S201031MS02Q
- removed U2: SeeeduinoXIAO, kicad_footprint-library-engg3800-alvin:Seeeduino XIAO-MOUDLE14P-2.54-21X17.8MM, symbol Seeeduino XIAO:SeeeduinoXIAO
- added J13: Conn_01x04_Pin, Connector_PinHeader_2.54mm:PinHeader_1x04_P2.54mm_Vertical, symbol Connector:Conn_01x04_Pin
Connections:
- net +3V3: now also J13.4 (Pin_4)
- net GND: now also J13.1 (Pin_1)
- net STM_RX: now also J13.2 (Pin_2)
- net STM_TX: now also J13.3 (Pin_3)
- no-connect marks 18 -> 2
Other:
- note removed: "10uF 10% 16V X5R"
- note removed: "SeeduinoXIAO"
