File: Sensor_Unit/peripherals.kicad_sch (KiCad schematic)
At the start: 41 parts, among them SW3 1825910-6, U14 CD74HCT164E, U15 CD74HCT164E

Commit message: Week 11 Sensor Unit Final Design - Submitted to Pinecone
Changed lines of the file:
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@@
 		(color 0 0 0 0)
 	)
-	(bus_entry
-		(at 43.18 31.75)
-		(size 2.54 2.54)
-		(stroke
-			(width 0)
-			(type default)
-		)
-	)
-	(bus_entry
-		(at 43.18 26.67)
-		(size 2.54 2.54)
-		(stroke
-			(width 0)
-			(type default)
-		)
-	)
 	(wire
 		(pts
@@
 	(wire
 		(pts
-			(xy 45.72 29.21) (xy 48.26 29.21)
-		)
-		(stroke
-			(width 0)
-			(type default)
-		)
-	)
-	(wire
-		(pts
 			(xy 53.34 78.74) (xy 67.31 78.74)
 		)
@@
 	(wire
 		(pts
-			(xy 45.72 34.29) (xy 48.26 34.29)
-		)
-		(stroke
-			(width 0)
-			(type default)
-		)
-	)
-	(wire
-		(pts
 			(xy 39.37 148.59) (xy 43.18 148.59)
 		)
@@
 		(pts
 			(xy 123.19 146.05) (xy 133.35 146.05)
-		)
-		(stroke
-			(width 0)
-			(type default)
-		)
-	)
-	(bus
-		(pts
-			(xy 43.18 22.86) (xy 39.37 22.86)
 		)
 		(stroke
@@
 		)
 	)
-	(bus
-		(pts
-			(xy 43.18 26.67) (xy 43.18 22.86)
-		)
-		(stroke
-			(width 0)
-			(type default)
-		)
-	)
 	(wire
 		(pts
@@
 		(pts
 			(xy 215.9 144.78) (xy 215.9 148.59)
-		)
-		(stroke
-			(width 0)
-			(type default)
-		)
-	)
-	(bus
-		(pts
-			(xy 43.18 31.75) (xy 43.18 26.67)
 		)
 		(stroke
@@
 		)
 	)
-	(hierarchical_label "ALARM_LED_ARRAYS"
-		(shape bidirectional)
-		(at 39.37 22.86 180)
-		(effects
-			(font
-				(size 1.27 1.27)
-			)
-			(justify right)
-		)
-	)
