File: Sensor_Unit/range_switching.kicad_sch (KiCad schematic)
At the start: 16 parts, among them J12 Conn_01x04_Pin, U18 DG509BEY-T1-E3, U19 TL072, U20 TL072, U21 AD5262BRUZ50

Commit message: Week 11 Sensor Unit Final Design - Submitted to Pinecone
Parts:
- added TP11: MUX_OUT, TestPoint:TestPoint_Loop_D2.54mm_Drill1.5mm_Beaded, symbol Connector:TestPoint
- added TP12: HALF_AT, TestPoint:TestPoint_Loop_D2.54mm_Drill1.5mm_Beaded, symbol Connector:TestPoint
- added TP13: DIFF, TestPoint:TestPoint_Loop_D2.54mm_Drill1.5mm_Beaded, symbol Connector:TestPoint
- added TP14: OFFSET_OUT, TestPoint:TestPoint_Loop_D2.54mm_Drill1.5mm_Beaded, symbol Connector:TestPoint
- added TP15: POT_A1, TestPoint:TestPoint_Loop_D2.54mm_Drill1.5mm_Beaded, symbol Connector:TestPoint
- added TP16: POT_W1, TestPoint:TestPoint_Loop_D2.54mm_Drill1.5mm_Beaded, symbol Connector:TestPoint
- added TP17: POT_A2, TestPoint:TestPoint_Loop_D2.54mm_Drill1.5mm_Beaded, symbol Connector:TestPoint
- added TP18: POT_W2, TestPoint:TestPoint_Loop_D2.54mm_Drill1.5mm_Beaded, symbol Connector:TestPoint
Connections:
- net POT_1B: now also TP13.1
- net POT_1W: now also TP16.1
- net POT_2W: now also TP18.1
- net at CR1.1, J12.2 (Pin_2), R58.2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: now also TP14.1
- net at R50.1, U18.8 (DA): now also TP11.1
- net at R52.2, R53.1, U19.1: now also TP12.1
- net at U21.16 (A2): now also TP17.1
- net at U21.2 (A1): now also TP15.1
- no-connect marks 8 -> 6
