File: Sensor_Unit/sensor_mcu.kicad_sch (KiCad schematic)
At the start: 11 parts, among them U1 STM32L431RCT6

Commit message: Week 11 Sensor Unit Final Design - Submitted to Pinecone
Parts:
- added FID1, FID2, FID3, FID4: Fiducial, kicad_footprint-library-engg3800-alvin:Fiducial_3mm_Mask6mm_custom_reuben, symbol Mechanical:Fiducial
- added R59: 10K 1% 0.100W, Resistor_THT:R_Axial_DIN0207_L6.3mm_D2.5mm_P10.16mm_Horizontal, symbol Device:R_US
Connections:
- net SPI_MISO_WEAK is gone; now on net SPI_MISO: R3.2
- net SPI_SCK is gone; now on net SPI_SCK_: R1.1
- net +3V3: now also U1.13 (VDDA)
- net GND: now also R59.1; no longer U1.13 (VDDA)
- net SPI_MISO: no longer R3.1
- net SPI_MOSI: no longer R2.1
- net SPI_SCK_: now reaches U1.15 (PA1)
- net SPI_MISO_: now reaches U1.22 (PA6)
- net SPI_MISO_: now also R3.1
- net at U1.60 (PH3): now also R59.2
- net JLink_SW0 renamed JLink_SWO
- net SCK renamed SPI_MOSI_
- net SPI_MOSI_: now also R2.1
- no-connect marks 0 -> 30
Other:
- moved on the sheet: C6, C7
