File: Sensor_Unit/voltage_channel_buffers.kicad_sch (KiCad schematic)
At the start: 6 parts, among them J10 Screw_Terminal_01x02, J11 Screw_Terminal_01x02, J8 Screw_Terminal_01x02, J9 Screw_Terminal_01x02, U16 TL072, U17 TL072

Commit message: Week 11 Sensor Unit Final Design - Submitted to Pinecone
Connections:
- net GND: now also J10.1, J11.1, J8.1, J9.1; no longer J10.2, J11.2, J8.2, J9.2
- net at U16.3 (+): now also J8.2; no longer J8.1
- net at U17.3 (+): now also J10.2; no longer J10.1
- net at U17.5 (+): now also J11.2; no longer J11.1
- net at U16.5 (+): now also J9.2; no longer J9.1
Other:
- moved on the sheet: J10, J11, J8, J9
