File: Control_Unit/Control_Unit_Final.kicad_sch (KiCad schematic)
At the start: 0 parts

Commit message: Final Control Unit Schematic Rev 1.
Other:
- added sheet Mechanicals (Mechanicals_sch.kicad_sch)
- sheet Joy and Sd and LCD ports: added DISPLAY, JOYSTICK, SD_CARD; removed none
- sheet MCU ports: added DISPLAY, JLINK, JOYSTICK, OPTIC_LINK, SD_CARD, XIAO; removed none
- sheet Optical Link ports: added OPTIC_LINK; removed none
- sheet Xiao and JLink ports: added JLINK, XIAO; removed none
- title: (none) -> ENGG3800 Team 03: Loggy
