File: Control_Unit/Main_Control_Unit.kicad_sch (KiCad schematic)
At the start: 12 parts, among them U1 STM32L431RCT6, Y1 AB26T-32.768KHZ

Commit message: Control Unit Schematics and PCB.
Parts:
- added FID1, FID2, FID3, FID4, FID5, FID6: Fiducial, kicad_footprint-library-engg3800-alvin:Fiducial_3mm_Mask6mm_custom_reuben, symbol Mechanical:Fiducial
- added R22: 10K, Resistor_THT:R_Axial_DIN0207_L6.3mm_D2.5mm_P10.16mm_Horizontal, symbol Device:R_US
Connections:
- net +3V3: now also U1.13 (VDDA)
- net GND: now also R22.1; no longer U1.13 (VDDA)
- net at U1.60 (PH3): now also R22.2
- net Button_Down renamed Btn_Down
- net Button_Left renamed Btn_Left
- net Button_Push renamed Btn_Push
- net Button_Right renamed Btn_Right
- net Button_Up renamed Btn_Up
- no-connect marks 29 -> 28
Other:
- moved on the sheet: C6, C7

Commit message: Final Control Unit Schematic Rev 1.
Parts:
- removed BT1: BHX1-2032-SM, kicad_footprint-library-engg3800-alvin:BAT_BHX1-2032-SM, symbol Earr_loggy_sym_lib:BHX1-2032-SM
- removed FID1, FID2, FID3, FID4, FID5, FID6: Fiducial, kicad_footprint-library-engg3800-alvin:Fiducial_3mm_Mask6mm_custom_reuben, symbol Mechanical:Fiducial
Connections:
- net +3V: now reaches U1.1 (VBAT)
- net Btn_Down renamed BTN_DOWN
- net Btn_Left renamed BTN_LEFT
- net Btn_Push renamed BTN_PUSH
- net Btn_Right renamed BTN_RIGHT
- net Btn_Up renamed BTN_UP
- net JLink_CLK renamed JLINK_CLK
- net JLink_RST renamed JLINK_RST
- net JLink_SW0 renamed JLINK_SW0
- net JLink_SWDIO renamed JLINK_SWDIO
Other:
- note added: "MCU"
- note added: "Peripheral Connections"
- title: (none) -> ENGG3800 Team 03: Loggy
- moved on the sheet: C1, C2, C3, C4, C5, C6, C7, C8, C9, R22, U1, Y1
