File: Control_Unit/Peripherals_sch.kicad_sch (KiCad schematic)
At the start: 7 parts, among them SW3 1825910-6

Commit message: Final Control Unit Schematic Rev 1.
Parts:
- R11: value 1K 1% 0W125 100R -> 1K/ 1%/ 0W125/ 100R
- R12: value 20R 1% 0.100W -> 20R/ 1%/ 0W100
- R13: value 62R 5% 0.100W -> 62R /5%/ 0W100
Other:
- note added: "Reset Swtich"
- note removed: "Reset Switch"
- title: (none) -> ENGG3800 Team 03: Loggy
- moved on the sheet: C17, LED1, LED2, R11, R12, R13, SW3
