File: Control_Unit/Xiao_and_JLink.kicad_sch (KiCad schematic)
At the start: 6 parts, among them J1 ETSG: 07-20-01, SW1 S201031MS02Q, U2 SeeeduinoXIAO

Commit message: Control Unit Schematics and PCB.
Parts:
- added TP1, TP2: TestPoint, TestPoint:TestPoint_Loop_D2.54mm_Drill1.5mm_Beaded, symbol Connector:TestPoint
Connections:
- net JLink_SWO is gone; now on net JLink_SW0: J1.8 (SWO)
- net +3V3: now also TP2.1
- net +5V: now also TP1.1
- no-connect marks 18 -> 19

Commit message: Final Control Unit Schematic Rev 1.
Parts:
- added TP3: TestPoint, symbol Connector:TestPoint
- D1: value 7.5V 500mW 5% -> 7.5V/ 500mW/ 5%
- TP1, TP2: footprint TestPoint:TestPoint_Loop_D2.54mm_Drill1.5mm_Beaded -> (none)
Connections:
- net GND: now also TP3.1
- net JLink_CLK renamed JLINK_CLK
- net JLink_RST renamed JLINK_RST
- net JLink_SW0 renamed JLINK_SW0
- net JLink_SWDIO renamed JLINK_SWDIO
Other:
- note added: "JLink Header"
- note added: "Seeduino Xiao"
- note added: "Test Points"
- note removed: "JLink"
- note removed: "SeeduinoXIAO"
- title: (none) -> ENGG3800 Team 03: Loggy
- moved on the sheet: C10, C11, D1, J1, SW1, U2
